File: board/WirelessTempSensor.brd (EAGLE design)
At the start: 41.9 x 17.8 mm, 16 parts, among them IC1 ATMEGA328P-AU, IC2 MCP9808, J1 PINHD-1X4, J2 PINHD-1X4, U1 MCP1700-3.0V, X1 SCREW-TERM-2

Commit message: Update BOM with more common value for R2
Parts:
- R2: value 150R -> 330R
Changed lines of the file:
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@@
 <?xml version="1.0" encoding="utf-8"?>
 <!DOCTYPE eagle SYSTEM "eagle.dtd">
-<eagle version="7.5.0">
+<eagle version="8.6.3">
 <drawing>
 <settings>
 <setting alwaysvectorfont="no"/>
+<setting keepoldvectorfont="yes"/>
 <setting verticaltext="up"/>
 </settings>
@@
 <param name="dpMaxLengthDifference" value="10mm"/>
 <param name="dpGapFactor" value="2.5"/>
-<param name="checkGrid" value="0"/>
 <param name="checkAngle" value="0"/>
 <param name="checkFont" value="1"/>
 <param name="checkRestrict" value="1"/>
+<param name="checkStop" value="0"/>
+<param name="checkValues" value="0"/>
 <param name="useDiameter" value="13"/>
 <param name="maxErrors" value="50"/>
@@
 <attribute name="NAME" x="30.988" y="16.3195" size="0.8128" layer="25"/>
 </element>
-<element name="R2" library="SaintGimp" package="RESISTOR-0805" value="150R" x="34.925" y="13.97" smashed="yes" rot="R90">
+<element name="R2" library="SaintGimp" package="RESISTOR-0805" value="330R" x="34.925" y="13.97" smashed="yes" rot="R90">
 <attribute name="NAME" x="34.163" y="16.3195" size="0.8128" layer="25"/>
 </element>
